Commit message: update b2z1_description

File: b2z1_description/urdf/b2z1.urdf (robot description, URDF)
Before this commit: robot b2z1_description, 47 links, 46 joints
Links:
- link FL_calf: mass 0.58094 -> 0.404; geometry collision box size=0.05 0.028 0.035; collision box size=0.1 0.0245 0.018
- link FL_foot: mass 0.098183 -> 0.126
- link FL_hip: mass 2.256 -> 2.673; geometry collision cylinder length=0.05 radius=0.07; visual mesh filename=package://b2z1_description/meshes/FL_hip.stl
- link FL_thigh: mass 3.591 -> 4.536; geometry collision box size=0.32 0.0445 0.054; visual mesh filename=package://b2z1_description/meshes/FL_thigh.stl
- link FR_calf: mass 0.58094 -> 0.404; geometry collision box size=0.05 0.028 0.035; collision box size=0.1 0.0245 0.018
- link FR_foot: mass 0.098183 -> 0.126
- link FR_hip: mass 2.256 -> 2.673; geometry collision cylinder length=0.05 radius=0.07; visual mesh filename=package://b2z1_description/meshes/FR_hip.stl
- link FR_thigh: mass 3.591 -> 4.536; geometry collision box size=0.25 0.028 0.04; visual mesh filename=package://b2z1_description/meshes/FR_thigh.stl
- link RL_calf: mass 0.58094 -> 0.404; geometry collision box size=0.05 0.028 0.035; collision box size=0.1 0.0245 0.018
- link RL_foot: mass 0.098183 -> 0.126
- link RL_hip: mass 2.256 -> 2.673; geometry collision cylinder length=0.05 radius=0.07; visual mesh filename=package://b2z1_description/meshes/RL_hip.stl
- link RL_thigh: mass 3.591 -> 4.536; geometry collision box size=0.25 0.028 0.04; visual mesh filename=package://b2z1_description/meshes/RL_thigh.stl
- link RR_calf: mass 0.58094 -> 0.404; geometry collision box size=0.05 0.028 0.035; collision box size=0.1 0.0245 0.018
- link RR_foot: mass 0.098183 -> 0.126
- link RR_hip: mass 2.256 -> 2.673; geometry collision cylinder length=0.05 radius=0.07; visual mesh filename=package://b2z1_description/meshes/RR_hip.stl
- link RR_thigh: mass 3.591 -> 4.536; geometry collision box size=0.25 0.028 0.04; visual mesh filename=package://b2z1_description/meshes/RR_thigh.stl
- link base_link: mass 35.606 -> 35.86; geometry collision box size=0.5 0.28 0.15; visual mesh filename=package://b2z1_description/meshes/base_link.stl
- link f_dc_link: mass 6.54E-08 -> 4.19E-15
- link f_oc_link: mass 6.55E-08 -> 4.19E-15
- link gripperMover: geometry collision mesh filename=package://b2z1_description/meshes/z1_GripperMover.obj scale=1 1 1; visual mesh filename=package://b2z1_description/meshes/z1_GripperMover.stl scale=1 1 1
- link gripperStator: geometry collision mesh filename=package://b2z1_description/meshes/z1_GripperStator.obj scale=1 1 1; visual mesh filename=package://b2z1_description/meshes/z1_GripperStator.stl scale=1 1 1
- link head_Link: mass 3.366 -> 3.6885
- link imu_link: mass 6.54E-08 -> 4.19E-15
- link lidar_link: mass 6.55E-08 -> 4.19E-15
- link link00: geometry collision cylinder length=0.051 radius=0.0325; visual mesh filename=package://b2z1_description/meshes/z1_Link00.stl scale=1 1 1
- link link01: geometry visual mesh filename=package://b2z1_description/meshes/z1_Link01.stl scale=1 1 1
- link link02: geometry collision cylinder length=0.051 radius=0.0325; collision cylinder length=0.102 radius=0.0325
- link link03: geometry collision cylinder length=0.059 radius=0.0325; collision cylinder length=0.116 radius=0.02
- link link04: geometry collision cylinder length=0.073 radius=0.0325; visual mesh filename=package://b2z1_description/meshes/z1_Link04.stl scale=1 1 1
- link link05: geometry visual mesh filename=package://b2z1_description/meshes/z1_Link05.stl scale=1 1 1
- link link06: geometry collision cylinder length=0.051 radius=0.0325; visual mesh filename=package://b2z1_description/meshes/z1_Link06.stl scale=1 1 1
- link r_dc_link: mass 6.55E-08 -> 4.19E-15
- link r_oc_link: mass 6.55E-08 -> 4.19E-12
- link tail_link: mass 0.777 -> 0.795
